File: uniKeyPCB.kicad_pcb (KiCad board)
At the start: 2 copper layers, 84 x 84 mm, 136 parts, among them J1 Conn_01x03_Socket, J10 Conn_01x02_Socket, J2 Conn_01x03_Socket, J3 Conn_01x02_Socket, J4 Conn_01x02_Socket, J5 Conn_01x03_Socket, J6 Conn_01x03_Socket, J9 Conn_01x02_Socket, SW1 SW_CHOC_HS, SW2 SW_MX_HS

Commit message: amended PCB
Other:
- board text added: "GND"
- board text added: "VCC"
