File: kicad/uniKeyPCB.kicad_sch (KiCad schematic)
At the start: 14 parts, among them J1 Conn_01x03_Socket, J10 Conn_01x02_Socket, J2 Conn_01x03_Socket, J3 Conn_01x02_Socket, J4 Conn_01x02_Socket, J5 Conn_01x03_Socket, J6 Conn_01x03_Socket, J9 Conn_01x02_Socket, SW1 SW_CHOC_HS, SW2 SW_MX_HS

Commit message: Silkscreen (#3)
* fixed silkscreen

* updaet screenshot
Parts:
- renumbered J5 to J3, J6 to J4, J9 to J5, J3 to J6, J10 to J7, J4 to J8
Changed lines of the file:
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@@
 		(on_board yes)
 		(dnp no)
-		(property "Reference" "J10"
+		(property "Reference" "J7"
 			(at 193.294 123.444 0)
 			(effects
@@
 			(project "uniKeyPCB"
 				(path "/b6ac1300-7796-4ba8-aab9-5215f43608b4"
-					(reference "J10")
+					(reference "J7")
 					(unit 1)
 				)
@@
 		(on_board yes)
 		(dnp no)
-		(property "Reference" "J6"
+		(property "Reference" "J4"
 			(at 240.919 90.17 0)
 			(effects
@@
 			(project "uniKeyPCB"
 				(path "/b6ac1300-7796-4ba8-aab9-5215f43608b4"
-					(reference "J6")
+					(reference "J4")
 					(unit 1)
 				)
@@
 		(on_board yes)
 		(dnp no)
-		(property "Reference" "J3"
+		(property "Reference" "J6"
 			(at 257.048 113.792 0)
 			(effects
@@
 			(project "uniKeyPCB"
 				(path "/b6ac1300-7796-4ba8-aab9-5215f43608b4"
-					(reference "J3")
+					(reference "J6")
 					(unit 1)
 				)
@@
 		(on_board yes)
 		(dnp no)
-		(property "Reference" "J4"
+		(property "Reference" "J8"
 			(at 257.048 123.444 0)
 			(effects
@@
 			(project "uniKeyPCB"
 				(path "/b6ac1300-7796-4ba8-aab9-5215f43608b4"
-					(reference "J4")
+					(reference "J8")
 					(unit 1)
 				)
@@
 		(on_board yes)
 		(dnp no)
-		(property "Reference" "J9"
+		(property "Reference" "J5"
 			(at 193.294 113.792 0)
 			(effects
@@
 			(project "uniKeyPCB"
 				(path "/b6ac1300-7796-4ba8-aab9-5215f43608b4"
-					(reference "J9")
+					(reference "J5")
 					(unit 1)
 				)
@@
 		(dnp no)
 		(fields_autoplaced yes)
-		(property "Reference" "J5"
+		(property "Reference" "J3"
 			(at 200.66 81.534 0)
 			(effects
@@
 			(project "uniKeyPCB"
 				(path "/b6ac1300-7796-4ba8-aab9-5215f43608b4"
-					(reference "J5")
-					(unit 1)
-				)
+					(reference "J3")
+					(unit 1)
+				)

Commit message: more connectors
Parts:
- added J10, J11, J12, J9: Conn_01x03_Socket, Connector_PinHeader_2.00mm:PinHeader_1x03_P2.00mm_Vertical, symbol Connector:Conn_01x03_Socket
- added J13, J14: Conn_01x02_Socket, Connector_PinSocket_2.00mm:PinSocket_1x02_P2.00mm_Vertical, symbol Connector:Conn_01x02_Socket
Connections:
- net GND: now also J13.1 (Pin_1), J14.1 (Pin_1)
- net LED0_in: now also J9.2 (Pin_2)
- net LED0_out: now also J10.2 (Pin_2)
- net LED1_in: now also J11.2 (Pin_2)
- net LED1_out: now also J12.2 (Pin_2)
- net VCC: now also J13.2 (Pin_2), J14.2 (Pin_2)
- net col0: now also J10.1 (Pin_1), J9.1 (Pin_1)
- net col1: now also J11.1 (Pin_1), J12.1 (Pin_1)
- net row0: now also J10.3 (Pin_3), J9.3 (Pin_3)
- net row1: now also J11.3 (Pin_3), J12.3 (Pin_3)
Other:
- moved on the sheet: J5, J6, J7, J8

Commit message: Revert "more connectors (#4)"
This reverts commit e986b9c313ce46b497b00528d1270ea63e1c5e11.
Parts:
- removed J10, J11, J12, J9: Conn_01x03_Socket, Connector_PinHeader_2.00mm:PinHeader_1x03_P2.00mm_Vertical, symbol Connector:Conn_01x03_Socket
- removed J13, J14: Conn_01x02_Socket, Connector_PinSocket_2.00mm:PinSocket_1x02_P2.00mm_Vertical, symbol Connector:Conn_01x02_Socket
Other:
- moved on the sheet: J5, J6, J7, J8
